Commit message: moveit_servo can now affect ar3 in webots simulation on

File: ar3/sim/config/ar2.urdf (robot description, URDF)
Before this commit: robot ar2, 7 links, 6 joints
Links:
- added link map
- link base_link: geometry collision mesh filename=file:///volume/meshes/base_link.STL; visual mesh filename=file:///volume/meshes/base_link.STL
- link link_1: geometry collision mesh filename=file:///volume/meshes/link_1.STL; visual mesh filename=file:///volume/meshes/link_1.STL
- link link_2: geometry collision mesh filename=file:///volume/meshes/link_2.STL; visual mesh filename=file:///volume/meshes/link_2.STL
- link link_3: geometry collision mesh filename=file:///volume/meshes/link_3.STL; visual mesh filename=file:///volume/meshes/link_3.STL
- link link_4: geometry collision mesh filename=file:///volume/meshes/link_4.STL; visual mesh filename=file:///volume/meshes/link_4.STL
- link link_5: geometry collision mesh filename=file:///volume/meshes/link_5.STL; visual mesh filename=file:///volume/meshes/link_5.STL
- link link_6: geometry collision mesh filename=file:///volume/meshes/link_6.STL; visual mesh filename=file:///volume/meshes/link_6.STL
Joints:
- added joint fixed: type fixed, parent map, child base_link
