Commit message: Updated PCB silk for AR3 breakout, worked on AR3 claw URDF file and visualization for it

File: ar3/sim/config/claw.urdf (robot description, URDF)
Before this commit: robot 2claw, 7 links, 6 joints
Links:
- link base: geometry visual mesh filename=file:///volume/meshes/Base_AR2.stl scale=0.001 0.001 0.001
- link claw1: geometry visual mesh filename=file:///volume/meshes/Claw.stl scale=0.001 0.001 0.001
- link claw2: geometry visual mesh filename=file:///volume/meshes/Claw.stl scale=0.001 0.001 0.001
- link con1: geometry visual mesh filename=file:///volume/meshes/Connector.stl scale=0.001 0.001 0.001
- link con2: geometry visual mesh filename=file:///volume/meshes/Connector.stl scale=0.001 0.001 0.001
- link congear1: geometry visual mesh filename=file:///volume/meshes/Connector_Gear.stl scale=0.001 0.001 0.001
- link congear2: geometry visual mesh filename=file:///volume/meshes/Servo_Connector_Gear.stl scale=0.001 0.001 0.001
Joints:
- joint joint1: axis (none) -> 0 0 1; limit (none) -> lower=-3.14 upper=3.14 effort=100 velocity=1.0; origin (none) -> xyz=0 0 0 rpy=0 0 0
- joint joint1mimic: limit (none) -> lower=-3.14 upper=3.14 effort=100 velocity=1.0
- joint joint2: limit (none) -> lower=-3.14 upper=3.14 effort=100 velocity=1.0
- joint joint2mimic: limit (none) -> lower=-3.14 upper=3.14 effort=100 velocity=1.0
- joint joint3: limit (none) -> lower=-3.14 upper=3.14 effort=100 velocity=1.0
- joint joint4: limit (none) -> lower=-3.14 upper=3.14 effort=100 velocity=1.0
